Commit message: made urdf model work in train package

File: urdf/train.urdf.xacro (robot description, xacro)
@@ -1,5 +1,5 @@
 <?xml version="1.0"?>
 <robot xmlns:xacro="http://www.ros.org/wiki/xacro" name="train">
-	<xacro:include filename="$(find turtlebot_description)/urdf/train/leg.urdf.xacro"/>
+	<xacro:include filename="$(find train)/urdf/train/leg.urdf.xacro"/>
 	<xacro:property name="width" value=".3" />
 	<xacro:property name="length" value=".4" />
@@ -7,4 +7,6 @@
 	<xacro:property name="wheeldiam" value=".07" />
 	<xacro:property name="M_PI" value="3.14159265" />
+	<xacro:property name="leg" value=".117" />
+        <xacro:property name="lowleg" value=".041" />
 <xacro:macro name="train">
  <link name="base_footprint"/>
@@ -47,5 +49,5 @@
   <axis xyz="0 -1 0"/>
   <limit effort="1000.0" lower="0" upper="6.28318" velocity="0.5"/>
-  <origin rpy="0 -${leg_angle} 0" xyz="${length/2} 0 0"/>
+  <origin rpy="0 -${leg_angle} 0" xyz="${.255/2} 0 0"/>
   <parent link="base_link"/>
   <child link="front_axle"/>
@@ -63,12 +65,12 @@
   <axis xyz="0 1 0"/>
   <limit effort="1000.0" lower="0" upper="6.28318" velocity="0.5"/>
-  <origin rpy="0 ${leg_angle} 0" xyz="-${length/2} 0 0"/>
+  <origin rpy="0 ${leg_angle} 0" xyz="-${.272/2} 0 0"/>
   <parent link="base_link"/>
   <child link="rear_axle"/>
  </joint>
-<xacro:leg prefix="front" suffix="right" leg_y="${width/2}" reflect="-1"/>
-<xacro:leg prefix="front" suffix="left" leg_y="-${width/2}" reflect="-1"/>
-<xacro:leg prefix="rear" suffix="right" leg_y="${width/2}" reflect="1"/>
-<xacro:leg prefix="rear" suffix="left" leg_y="-${width/2}" reflect="1"/>
+<xacro:leg prefix="front" suffix="right" leg_y="1" reflect="-1"/>
+<xacro:leg prefix="front" suffix="left" leg_y="-1" reflect="-1"/>
+<xacro:leg prefix="rear" suffix="right" leg_y="1" reflect="1"/>
+<xacro:leg prefix="rear" suffix="left" leg_y="-1" reflect="1"/>
 </xacro:macro>
 </robot>

File: urdf/train/leg.urdf.xacro (robot description, xacro)
@@ -5,7 +5,7 @@
   <visual>
    <geometry>
-    <box size="0.02 .05 .1"/>
+    <box size="0.05 .05 ${leg}"/>
    </geometry>
-   <origin rpy="0 0 0" xyz="0.0 0.0 0.05"/>
+   <origin rpy="0 0 0" xyz="0.0 0.0 ${leg/2}"/>
    <material name="white">
     <color rgba="1 1 1 1"/>
@@ -15,5 +15,5 @@
  <joint name="base_to_${prefix}_${suffix}_leg" type="fixed">
   <axis xyz="1 0 0"/>
-  <origin rpy="0 3.1415 1.57075" xyz="0 ${leg_y} 0"/>
+  <origin rpy="0 3.1415 1.57075" xyz="0 ${leg_y*((width/2)+0.025)} 0"/>
   <parent link="${prefix}_axle"/>
   <child link="${prefix}_${suffix}_leg"/>
@@ -22,7 +22,7 @@
   <visual>
    <geometry>
-    <box size="0.02 .05 .05"/>
+    <box size="0.04 .05 ${lowleg}"/>
    </geometry>
-   <origin rpy="0 0 0" xyz="0.0 0.0 0.025"/>
+   <origin rpy="0 0 0" xyz="0.0 0.0 ${lowleg/2}"/>
    <material name="white"/>
   </visual>
@@ -31,5 +31,5 @@
   <axis xyz="${reflect} 0 0"/>
   <limit effort="1000.0" velocity="0.5"/>
-  <origin rpy="0 0 0" xyz="0.0 0.0 0.1"/>
+  <origin rpy="0 0 0" xyz="${leg_y*-1*0.04} 0.0 ${leg}"/>
   <parent link="${prefix}_${suffix}_leg"/>
   <child link="${prefix}_${suffix}_lowleg"/>
@@ -48,5 +48,5 @@
   <axis xyz="0 0 1"/>
   <limit effort="1000.0" lower="-3.1415" upper="3.1415" velocity="0.5"/>
-  <origin rpy="0 0 0" xyz="0.0 0.0 0.05"/>
+  <origin rpy="0 0 0" xyz="0.0 0.0 ${lowleg}"/>
   <parent link="${prefix}_${suffix}_lowleg"/>
   <child link="${prefix}_${suffix}_turnleg"/>
@@ -55,5 +55,5 @@
     <visual>
       <geometry>
-        <cylinder length=".05" radius="${wheeldiam/2}"/>
+        <mesh filename="package://train/urdf/meshes/hjul.stl" />
       </geometry>
       <material name="black">
