Commit message: reading leg-angles work

File: urdf/test.urdf (robot description, URDF)
Before this commit: robot train, 20 links, 19 joints
Joints:
- joint base_to_front_axle: limit lower=0 upper=6.28318 effort=1000.0 velocity=0.5 -> lower=-6.28318 upper=6.28318 effort=1000.0 velocity=0.5
- joint base_to_rear_axle: limit lower=0 upper=6.28318 effort=1000.0 velocity=0.5 -> lower=-6.28318 upper=6.28318 effort=1000.0 velocity=0.5
